File: kiCAD/_autosave-kiCAD Keypad.kicad_pcb (KiCad board)
At the start: 4 copper layers, 93.2 x 155.8 mm, 71 parts, among them J1 USB_C_Receptacle_USB2.0_16P, J3 2x8 GPIO for SPI, SW1 RESET, SW2 BOOT, SW3 RotaryEncoder_Switch, U1 ESP32-S3-WROOM-2, U2 USBLC6-2SC6, U3 MIC5365-3.3YD5

Commit message: Exporting to JLCPCB
Parts:
- removed U3: MIC5365-3.3YD5, Package_TO_SOT_SMD:SOT-23-5
- added U4: AP2112K-3.3, Package_TO_SOT_SMD:SOT-23-5, F.Cu at (64.8, 48.4)
- C3: value 1uF -> 0u1F
- moved U2 1.99 mm to (55.5, 47.4)
Routing:
- net GND: track 6.80 -> 14.7 mm
- net /5V_IN: track 32.5 -> 28.9 mm
- net /ESP32_D-: track 33.6 -> 35.5 mm
- net /ESP32_D+: track 36.7 -> 38.7 mm
- net /USBC_D-: track 9.95 -> 8.13 mm
- net /USBC_D+: track 8.67 -> 6.96 mm
