File: kiCAD/kiCAD Keypad.kicad_pcb (KiCad board)
At the start: 4 copper layers, 93.2 x 155.8 mm, 71 parts, among them J1 USB_C_Receptacle_USB2.0_16P, J3 2x8 GPIO for SPI, SW1 RESET, SW2 BOOT, SW3 RotaryEncoder_Switch, U1 ESP32-S3-WROOM-2, U2 USBLC6-2SC6, U3 MIC5365-3.3YD5

Commit message: Exporting to JLCPCB
Parts:
- removed U3: MIC5365-3.3YD5, Package_TO_SOT_SMD:SOT-23-5
- added U4: AP2112K-3.3, Package_TO_SOT_SMD:SOT-23-5, F.Cu at (64.8, 48.4)
- C3: value 1uF -> 0u1F
- moved U2 1.99 mm to (55.5, 47.4)
Routing:
- net GND: track 6.80 -> 14.7 mm
- net /5V_IN: track 32.5 -> 28.9 mm
- net /ESP32_D-: track 33.6 -> 35.5 mm
- net /ESP32_D+: track 36.7 -> 38.7 mm
- net /USBC_D-: track 9.95 -> 8.13 mm
- net /USBC_D+: track 8.67 -> 6.96 mm

Commit message: Iterating; deciding on switching to devkit
Parts:
- removed U1: ESP32-S3-WROOM-2, RF_Module:ESP32-S3-WROOM-2
- added J2: Conn_01x04, Connector_PinHeader_2.54mm:PinHeader_1x04_P2.54mm_Vertical, F.Cu at (122.3, 62.0)
- added U3: ESP32-S3-MINI-1, RF_Module:ESP32-S2-MINI-1, F.Cu at (91.5, 50.1)
- C3: footprint Capacitor_SMD:C_0805_2012Metric -> Capacitor_SMD:C_0402_1005Metric
- moved SW1 46.6 mm to (114.2, 48.7), turned to 90 degrees
- moved SW2 41.2 mm to (67.7, 54.6), turned to 90 degrees
- moved C3 38.8 mm to (110.0, 46.5), turned to -90 degrees
- moved R1 38.2 mm to (110.2, 49.9)
- moved C4 32.0 mm to (72.3, 55.6)
- moved R2 32.0 mm to (72.3, 53.5)
- moved D22 10.8 mm to (85.0, 62.8)
- moved R7 10.8 mm to (82.3, 62.8)
- moved C1 0.08 mm to (81.2, 47.9)
Routing:
- net /ESP32_TX: track 0.00 -> 27.0 mm
- net /ESP32_RX: track 0.00 -> 26.3 mm
- net /RE_B: track 36.8 -> 19.1 mm
- net /ESP32_D+: track 38.7 -> 54.7 mm
- net /ESP32_D-: track 35.5 -> 49.3 mm
- net /ESP32_BOOT: track 14.9 -> 25.6 mm
- net /RE_A: track 33.7 -> 25.0 mm
- net GND: track 14.7 -> 22.8 mm
- net /Row_5: track 191.2 -> 184.5 mm
- net /Row_4: track 193.4 -> 186.9 mm
- net /Row_3: track 169.2 -> 163.0 mm
- net /Row_2: track 146.4 -> 140.5 mm
- net /Row_1: track 124.5 -> 118.7 mm
- net /Row_0: track 103.5 -> 98.2 mm
- net /RE_SW: track 40.6 -> 35.8 mm
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